Commit message: Miniaturize Four Wheel Diff BS Robot for pig pen simulation (0.4m x 0.35m)

File: turn_on_wheeltec_robot/urdf/four_wheel_diff_bs_robot.urdf (robot description, URDF)
Before this commit: robot wheeltec_robot, 5 links, 4 joints
Links:
- added link laser_link, mass 0.2; collision cylinder length=0.05 radius=0.04; visual cylinder length=0.05 radius=0.04
- link base_link: mass None -> 15.0; geometry collision box size=0.4 0.35 0.150; visual box size=0.4 0.35 0.150
- link left_front_link: mass None -> 1.5; geometry collision cylinder length=0.04 radius=0.06; visual cylinder length=0.04 radius=0.06
- link left_wheel_link: mass None -> 1.5; geometry collision cylinder length=0.04 radius=0.06; visual cylinder length=0.04 radius=0.06
- link right_front_link: mass None -> 1.5; geometry collision cylinder length=0.04 radius=0.06; visual cylinder length=0.04 radius=0.06
- link right_wheel_link: mass None -> 1.5; geometry collision cylinder length=0.04 radius=0.06; visual cylinder length=0.04 radius=0.06
Joints:
- added joint laser_joint: type fixed, parent base_link, child laser_link, origin xyz=0.0 0 0.22 rpy=0 0 0
- joint left_front_joint: axis 0 1 0 -> 0 0 1; origin xyz=0.0 0.298 0.109 rpy=1.57 0 0 -> xyz=-0.05 0.20 0.06 rpy=-1.570796 0 0
- joint left_wheel_joint: axis 0 1 0 -> 0 0 1; origin xyz=-0.33 0.29 0.109 rpy=1.57 0 0 -> xyz=-0.22 0.20 0.06 rpy=-1.570796 0 0
- joint right_front_joint: axis 0 1 0 -> 0 0 1; origin xyz=0.0 -0.298 0.109 rpy=1.57 0 0 -> xyz=-0.05 -0.20 0.06 rpy=-1.570796 0 0
- joint right_wheel_joint: axis 0 1 0 -> 0 0 1; origin xyz=-0.33 -0.29 0.109 rpy=1.57 0 0 -> xyz=-0.22 -0.20 0.06 rpy=-1.570796 0 0

Commit message: Fix robot dimensions to 0.45(L) x 0.4(W)

File: turn_on_wheeltec_robot/urdf/four_wheel_diff_bs_robot.urdf (robot description, URDF)
Before this commit: robot wheeltec_robot, 6 links, 5 joints
Links:
- link base_link: geometry collision box size=0.45 0.4 0.150; visual box size=0.45 0.4 0.150
Joints:
- joint left_front_joint: origin xyz=-0.05 0.20 0.06 rpy=-1.570796 0 0 -> xyz=0.15 0.22 0.06 rpy=-1.570796 0 0
- joint left_wheel_joint: origin xyz=-0.22 0.20 0.06 rpy=-1.570796 0 0 -> xyz=-0.15 0.22 0.06 rpy=-1.570796 0 0
- joint right_front_joint: origin xyz=-0.05 -0.20 0.06 rpy=-1.570796 0 0 -> xyz=0.15 -0.22 0.06 rpy=-1.570796 0 0
- joint right_wheel_joint: origin xyz=-0.22 -0.20 0.06 rpy=-1.570796 0 0 -> xyz=-0.15 -0.22 0.06 rpy=-1.570796 0 0

Commit message: fix(urdf): 修正 base_link 與感測器位置
Center base_link origin; center laser_joint; move depth camera to front edge.

File: turn_on_wheeltec_robot/urdf/four_wheel_diff_bs_robot.urdf (robot description, URDF)
Before this commit: robot wheeltec_robot, 6 links, 5 joints
Links:
- added link depth_camera_link, mass 0.2; collision box size=0.08 0.06 0.03; visual box size=0.08 0.06 0.03
- link base_link: geometry collision box size=0.67 0.53 0.150; visual box size=0.67 0.53 0.150
- link left_front_link: geometry collision cylinder length=0.04 radius=0.109; visual cylinder length=0.04 radius=0.109
- link left_wheel_link: geometry collision cylinder length=0.04 radius=0.109; visual cylinder length=0.04 radius=0.109
- link right_front_link: geometry collision cylinder length=0.04 radius=0.109; visual cylinder length=0.04 radius=0.109
- link right_wheel_link: geometry collision cylinder length=0.04 radius=0.109; visual cylinder length=0.04 radius=0.109
Joints:
- added joint depth_camera_joint: type fixed, parent base_link, child depth_camera_link, origin xyz=0.37 0 0.23 rpy=0 0 0
- joint laser_joint: origin xyz=0.0 0 0.22 rpy=0 0 0 -> xyz=0.0 0 0.26 rpy=0 0 0
- joint left_front_joint: axis 0 0 1 -> 0 0 -1; origin xyz=0.15 0.22 0.06 rpy=-1.570796 0 0 -> xyz=0.3 0.285 0.109 rpy=1.57 0 0
- joint left_wheel_joint: axis 0 0 1 -> 0 0 -1; origin xyz=-0.15 0.22 0.06 rpy=-1.570796 0 0 -> xyz=-0.3 0.285 0.109 rpy=1.57 0 0
- joint right_front_joint: axis 0 0 1 -> 0 0 -1; origin xyz=0.15 -0.22 0.06 rpy=-1.570796 0 0 -> xyz=0.3 -0.285 0.109 rpy=1.57 0 0
- joint right_wheel_joint: axis 0 0 1 -> 0 0 -1; origin xyz=-0.15 -0.22 0.06 rpy=-1.570796 0 0 -> xyz=-0.3 -0.285 0.109 rpy=1.57 0 0

Commit message: Update simulation pipeline and sync robot dimensions

File: turn_on_wheeltec_robot/urdf/four_wheel_diff_bs_robot.urdf (robot description, URDF)
Before this commit: robot wheeltec_robot, 7 links, 6 joints
Links:
- link base_link: geometry collision box size=0.40 0.30 0.165; visual box size=0.40 0.30 0.165
- link left_front_link: geometry collision cylinder length=0.05 radius=0.109; visual cylinder length=0.05 radius=0.109
- link left_wheel_link: geometry collision cylinder length=0.05 radius=0.109; visual cylinder length=0.05 radius=0.109
- link right_front_link: geometry collision cylinder length=0.05 radius=0.109; visual cylinder length=0.05 radius=0.109
- link right_wheel_link: geometry collision cylinder length=0.05 radius=0.109; visual cylinder length=0.05 radius=0.109
Joints:
- joint depth_camera_joint: origin xyz=0.37 0 0.23 rpy=0 0 0 -> xyz=0.2 0 0.095 rpy=0 0 0
- joint laser_joint: origin xyz=0.0 0 0.26 rpy=0 0 0 -> xyz=0.0 0 0.245 rpy=0 0 0
- joint left_front_joint: origin xyz=0.3 0.285 0.109 rpy=1.57 0 0 -> xyz=0.14 0.175 0.075 rpy=1.57 0 0
- joint left_wheel_joint: origin xyz=-0.3 0.285 0.109 rpy=1.57 0 0 -> xyz=-0.14 0.175 0.075 rpy=1.57 0 0
- joint right_front_joint: origin xyz=0.3 -0.285 0.109 rpy=1.57 0 0 -> xyz=0.14 -0.175 0.075 rpy=1.57 0 0
- joint right_wheel_joint: origin xyz=-0.3 -0.285 0.109 rpy=1.57 0 0 -> xyz=-0.14 -0.175 0.075 rpy=1.57 0 0

Commit message: 更新深度相機為ZEDX/更新雷達為自製模型參數參考M10P-PHY

File: turn_on_wheeltec_robot/urdf/four_wheel_diff_bs_robot.urdf (robot description, URDF)
Before this commit: robot wheeltec_robot, 7 links, 6 joints
Links:
- link depth_camera_link: mass 0.2 -> 0.25; geometry collision box size=0.175 0.03 0.04; visual box size=0.175 0.03 0.04
- link laser_link: geometry collision cylinder length=0.039 radius=0.0398; visual cylinder length=0.039 radius=0.0398
