Commit message: 新增隨機豬隻模型與小車右側相機

File: turn_on_wheeltec_robot/urdf/four_wheel_diff_bs_robot.urdf (robot description, URDF)
Before this commit: robot wheeltec_robot, 7 links, 6 joints
Links:
- added link right_camera_link, mass 0.1; collision box size=0.05 0.05 0.05; visual box size=0.05 0.05 0.05
Joints:
- added joint right_camera_joint: type fixed, parent base_link, child right_camera_link, origin xyz=0 -0.15 0.15 rpy=0 0 -1.5708
